File: Led-Controller.kicad_sch (KiCad schematic)
At the start: 31 parts, among them Q1 PMOS, Q2 PMOS, Q3 PMOS, Q4 PMOS, Q5 PMOS, U1 1ED44175N01BXTSA1, U2 1ED44175N01BXTSA1, U3 1ED44175N01BXTSA1, U4 1ED44175N01BXTSA1, U5 1ED44175N01BXTSA1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

Commit message: Final PCB
Parts:
- added C10, C11, C12, C13, C14, C15, C16, C17: C, Capacitor_SMD:C_0805_2012Metric_Pad1.18x1.45mm_HandSolder, symbol Device:C
- added J1: Barrel_Jack_Switch_Pin3Ring, Connector_BarrelJack:BarrelJack_GCT_DCJ200-10-A_Horizontal, symbol Connector:Barrel_Jack_Switch_Pin3Ring
- added J2: Screw_Terminal_01x06, TerminalBlock:TerminalBlock_bornier-6_P5.08mm, symbol Connector:Screw_Terminal_01x06
- added U8: AMS1117-5.0, Package_TO_SOT_SMD:SOT-223-3_TabPin2, symbol Regulator_Linear:AMS1117-5.0
- Q1, Q2, Q3, Q4, Q5: footprint MOSFETS:BSZ180P03 -> BSZ180P03:BSZ180P03
Connections:
- net GND: now also C10.2, C11.2, C12.2, C13.2, C14.2, C15.2, C16.2, C17.2, J1.2, J1.3, J2.1 (Pin_1), U8.1 (GND)
- net IN1: now also U6.13 (IO14)
- net IN2: now also U6.12 (IO27)
- net IN3: now also U6.11 (IO26)
- net IN4: now also U6.10 (IO25)
- net IN5: now also U6.9 (IO33)
- net VCC: now also C11.1, C12.1, C13.1, C14.1, C15.1, C16.1, C17.1, J1.1, U8.3 (VI); no longer C6.1, U7.3 (VI)
- net at Q4.1 (D): now also J2.3 (Pin_3)
- net at Q3.1 (D): now also J2.4 (Pin_4)
- net at Q5.1 (D): now also J2.2 (Pin_2)
- net at Q1.1 (D): now also J2.6 (Pin_6)
- net at Q2.1 (D): now also J2.5 (Pin_5)
- new net +5V: C10.1, C6.1, U7.3 (VI), U8.2 (VO)
